File: analog.kicad_sch (KiCad schematic)
At the start: 0 parts

Commit message: Schema devrait etre fini. A revalider avec le layout (Surtout SWO pour debug)
Parts:
- added C24, C25, C26, C27, C28, C29, C30, C31: 160n, Capacitor_SMD:C_0402_1005Metric_Pad0.74x0.62mm_HandSolder, symbol Device:C
- added R22, R24, R26, R28, R30, R32, R34, R36: 33k, Resistor_SMD:R_0603_1608Metric_Pad0.98x0.95mm_HandSolder, symbol Device:R_US
- added R23, R25, R27, R29, R31, R33, R35, R37: 50k, Resistor_SMD:R_0603_1608Metric_Pad0.98x0.95mm_HandSolder, symbol Device:R_US
Connections:
- new net GND: C24.2, C25.2, C26.2, C27.2, C28.2, C29.2, C30.2, C31.2, R23.2, R25.2, R27.2, R29.2, R31.2, R33.2, R35.2, R37.2
- new net analog_in0: R22.1
- new net analog_in0_filt: C24.1, R22.2, R23.1
- new net analog_in1: R24.1
- new net analog_in1_filt: C25.1, R24.2, R25.1
- new net analog_in2: R26.1
- new net analog_in2_filt: C26.1, R26.2, R27.1
- new net analog_in3: R28.1
- new net analog_in3_filt: C27.1, R28.2, R29.1
- new net analog_in4: R30.1
- new net analog_in4_filt: C28.1, R30.2, R31.1
- new net analog_in5: R32.1
- new net analog_in5_filt: C29.1, R32.2, R33.1
- new net analog_in6: R34.1
- new net analog_in6_filt: C30.1, R34.2, R35.1
- new net analog_in7: R36.1
- new net analog_in7_filt: C31.1, R36.2, R37.1
Other:
- note added: "Analog input filtering"
- note added: "Input cutoff frequency is 50 Hz Minimal sampling rate is 100 Hz"
